File: pcb/Hackpad.kicad_pcb (KiCad board)
At the start: 2 copper layers, 100 x 65 mm, 11 parts, among them J1 SSD1306 OLED, SW1 SW_Push, SW2 SW_Push, SW3 SW_Push, SW4 SW_Push, SW5 RotaryEncoder_Switch, U1 XIAO-RP2040-DIP

Commit message: pcb errors. fixed
Parts:
- added CyreneBack: LOGO, CyrenePad-Images:CyreneSilk, B.Cu at (100.3, 109.0)
- added CyreneLeft: LOGO, CyrenePad-Images:CyreneChibi1, F.Cu at (58.2, 103.4)
- added CyrenePeek: LOGO, CyrenePad-Images:CyrenePeeking, F.Cu at (79.8, 135.1)
- added CyreneRight: LOGO, CyrenePad-Images:CyrenePoint, F.Cu at (140.8, 103.7)
- added D5: SK6812MINI, PCM_marbastlib-mx:LED_MX_6028R, B.Cu at (128.0, 126.9)
- added D6: SK6812MINI, PCM_marbastlib-mx:LED_MX_6028R, B.Cu at (108.9, 126.9)
- added D7: SK6812MINI, PCM_marbastlib-mx:LED_MX_6028R, B.Cu at (89.9, 126.9)
- added D8: SK6812MINI, PCM_marbastlib-mx:LED_MX_6028R, B.Cu at (70.9, 126.8)
- D1, D2, D3, D4: footprint LED_SMD:LED_SK6812MINI_PLCC4_3.5x3.5mm_P1.75mm -> PCM_marbastlib-mx:LED_MX_6028R; moved to B.Cu
- turned D1 to 180 degrees
- turned D2 to 180 degrees
- turned D3 to 180 degrees
- turned D4 to 180 degrees
Connections:
- D4 pad 1: unconnected-(D4-DOUT-Pad1) -> Net-(D4-DOUT)
- J1 pad 1: Net-(J1-Pin_1) -> GND
- J1 pad 2: Net-(J1-Pin_2) -> VCC
- J1 pad 3: VCC -> Net-(J1-Pin_3)
- J1 pad 4: GND -> Net-(J1-Pin_4)
- SW5 pad S2: Net-(U1-GPIO29/ADC3/A3) -> GND
- U1 pad 12: unconnected-(U1-3V3-Pad12) -> VCC
- U1 pad 4: Net-(U1-GPIO29/ADC3/A3) -> Net-(D1-DIN)
- U1 pad 5: Net-(D1-DIN) -> Net-(J1-Pin_4)
- U1 pad 6: Net-(J1-Pin_1) -> Net-(J1-Pin_3)
- U1 pad 7: Net-(J1-Pin_2) -> unconnected-(U1-GPIO0/TX-Pad7)
Routing:
- net +5V: track 96.2 -> 189.6 mm, vias 1 -> 0
- net GND: track 215.6 -> 265.4 mm
- net Net-(J1-Pin_2): track 35.2 -> 0.00 mm
- net Net-(J1-Pin_4): track 0.00 -> 30.3 mm
- net Net-(J1-Pin_3): track 0.00 -> 29.5 mm
- net Net-(J1-Pin_1): track 28.1 -> 0.00 mm
- net Net-(D4-DOUT): track 0.00 -> 24.4 mm
- net Net-(D7-DOUT): track 0.00 -> 18.8 mm, vias 0 -> 2
- net Net-(D6-DOUT): track 0.00 -> 18.5 mm, vias 0 -> 2
- net Net-(D5-DOUT): track 0.00 -> 17.5 mm, vias 0 -> 2
- net VCC: track 0.00 -> 14.1 mm
- net Net-(U1-GPIO29/ADC3/A3): track 12.7 -> 0.00 mm
- net Net-(U1-GPIO1/RX): track 66.5 -> 57.1 mm
- net Net-(U1-GPIO3/MOSI): track 67.2 -> 59.0 mm
- net Net-(U1-GPIO2/SCK): track 35.7 -> 42.3 mm, vias 0 -> 1
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Other:
- outline, holes or cut-outs redrawn
- board text added: "PhiLia093 /// Ripples of Past Reverie /// Cyrene /// Elysia ///"
- board text added: "this will be a romantic story like none that has come before... you think so too, right?"
- board text added: "キュレネ Hackpad v2"
- board text removed: "キュレネ Hackpad v1"
