File: pcb/Hackpad.kicad_sch (KiCad schematic)
At the start: 11 parts, among them J1 SSD1306 OLED, SW1 SW_Push, SW2 SW_Push, SW3 SW_Push, SW4 SW_Push, SW5 RotaryEncoder_Switch, U1 XIAO-RP2040-DIP

Commit message: pcb errors. fixed
Parts:
- added D5, D6, D7, D8: SK6812MINI, PCM_marbastlib-mx:LED_MX_6028R, symbol LED:SK6812MINI
- D1, D2, D3, D4: footprint LED_SMD:LED_SK6812MINI_PLCC4_3.5x3.5mm_P1.75mm -> PCM_marbastlib-mx:LED_MX_6028R
Connections:
- net +5V: now also D5.4 (VDD), D6.4 (VDD), D7.4 (VDD), D8.4 (VDD)
- net GND: now also J1.1 (Pin_1), D5.2 (VSS), D6.2 (VSS), D7.2 (VSS), D8.2 (VSS); no longer J1.4 (Pin_4)
- net VCC: now also J1.2 (Pin_2), U1.12 (3V3); no longer J1.3 (Pin_3)
- net at U1.6 (GPIO7/SCL): now also J1.3 (Pin_3); no longer J1.1 (Pin_1)
- net at U1.7 (GPIO0/TX): no longer J1.2 (Pin_2)
- net at U1.4 (GPIO29/ADC3/A3): now also D1.3 (DIN)
- net at U1.5 (GPIO6/SDA): now also J1.4 (Pin_4); no longer D1.3 (DIN)
- net at D4.1 (DOUT): now also D5.3 (DIN)
- new net: D5.1 (DOUT), D6.3 (DIN)
- new net: D7.1 (DOUT), D8.3 (DIN)
- new net: D6.1 (DOUT), D7.3 (DIN)
Other:
- moved on the sheet: D1, D2, D3, D4
